File: Labs/lab7/lab7PCB/lab7.kicad_pcb (KiCad board)
At the start: 2 copper layers, 0 parts

Commit message: lab7: Leo PCB practice
Co-Authored-By: Claude Opus 5.5 <noreply@anthropic.com>
Other:
- board outline added: 63.5 x 63.5 mm
Changed lines of the file:
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@@
 		(capping no)
 		(filling no)
-		(zone_defaults)
 		(pcbplotparams
 			(layerselection 0x00000000_00000000_55555555_5755f5ff)
@@
 		)
 	)
+	(gr_rect
+		(start 90.75 55.75)
+		(end 154.25 119.25)
+		(stroke
+			(width 0.05)
+			(type default)
+		)
+		(fill no)
+		(layer "Edge.Cuts")
+	)
 	(embedded_fonts no)
