File: Labs/lab7/lab7PCB/lab7LeoPCBPractice.kicad_pcb (KiCad board)
At the start: 2 copper layers, 63.5 x 63.5 mm, 13 parts, among them SW1 SW_Vibe, SW2 SW_Push, U1 YD-ESP32-S3

Commit message: silkscreen fix
Routing:
- net Net-(U1-GPIO4): track 0.00 -> 84.3 mm
- net GND: track 0.00 -> 77.1 mm
- net Net-(U1-GPIO5): track 0.00 -> 74.1 mm
- net Net-(U1-GPIO6): track 0.00 -> 39.6 mm
- net Net-(R3-Pad1): track 0.00 -> 32.7 mm
- net Net-(U1-GPIO7): track 0.00 -> 20.9 mm
- net Net-(U1-GPIO8): track 0.00 -> 14.2 mm
- net Net-(D1-A): track 0.00 -> 5.36 mm
Other:
- board text added: "Hello World"

Commit message: silkscreen art
Parts:
- added G***: LOGO, LOGO, F.Cu at (124.0, -216.0)
